File: pcb/eightzero.kicad_pcb (KiCad board)
At the start: 2 copper layers, 155.6 x 90.6 mm, 13 parts, among them P1 ADDRESS, P2 DATA, P3 PORT_A, P4 PORT_B, P5 PORT_C, P6 PORT_D, P7 MII, U1 EZ80F91

Commit message: components, routing
Parts:
- added C1: ~, SM0402, F.Cu at (153.4, 82.0)
- added C2: ~, SM0402, F.Cu at (153.4, 86.0)
- added C3: ~, SM0402, F.Cu at (153.4, 90.0)
- added C4: ~, SM0402, F.Cu at (153.4, 94.5)
- added C5: ~, SM0402, F.Cu at (157.9, 101.0)
- added J1: VGA, EDAC_15, F.Cu at (199.5, 57.0)
- added R1: R, R4, F.Cu at (209.6, 67.7)
- added R2: R, R4, F.Cu at (207.1, 67.7)
- added R3: R, R4, F.Cu at (204.5, 67.7)
- added R4: R, R4, F.Cu at (202.0, 67.7)
- added R5: R, R4, F.Cu at (199.5, 67.7)
- added R6: R, R4, F.Cu at (196.9, 67.7)
- added R7: R, R4, F.Cu at (194.4, 67.7)
- added R8: R, R4, F.Cu at (191.8, 67.7)
- added R9: R, R4, F.Cu at (189.3, 67.7)
- added U2: GD_CORE, TQFP_100, F.Cu at (199.5, 85.5)
- P3: value PORT_A -> PORT A
- P4: value PORT_B -> PORT B
- P5: value PORT_C -> PORT C
- P6: value PORT_D -> PORT D
- moved P6 45.9 mm to (221.1, 126.1)
- moved P5 44.7 mm to (221.1, 108.3)
- moved P3 37.1 mm to (221.1, 72.8)
- moved P4 34.3 mm to (221.1, 90.6)
- moved P1 6.93 mm to (139.8, 81.7)
- moved P2 6.93 mm to (139.8, 117.2)
- moved U1 4.54 mm to (166.4, 88.0)
- moved P7 1.93 mm to (160.1, 61.4)
- moved Breadboard 0.85 mm to (115.6, 99.5)
Connections:
- U1 pad 108: (no net) -> GND
- U1 pad 112: (no net) -> +3.3V
- U1 pad 113: (no net) -> GND
- U1 pad 122: (no net) -> +3.3V
- U1 pad 123: (no net) -> GND
- U1 pad 133: (no net) -> +3.3V
- U1 pad 134: (no net) -> GND
- U1 pad 14: (no net) -> +3.3V
- U1 pad 15: (no net) -> GND
- U1 pad 22: (no net) -> +3.3V
- U1 pad 23: (no net) -> GND
- U1 pad 31: (no net) -> +3.3V
- U1 pad 32: (no net) -> GND
- U1 pad 37: (no net) -> +3.3V
- U1 pad 38: (no net) -> GND
- U1 pad 47: (no net) -> +3.3V
- U1 pad 48: (no net) -> GND
- U1 pad 59: (no net) -> +3.3V
- U1 pad 6: (no net) -> +3.3V
- U1 pad 60: (no net) -> GND
- U1 pad 64: (no net) -> GND
- U1 pad 7: (no net) -> GND
- U1 pad 72: (no net) -> GND
- U1 pad 81: (no net) -> +3.3V
- U1 pad 82: (no net) -> GND
- U1 pad 88: (no net) -> +3.3V
- U1 pad 89: (no net) -> GND
- U1 pad 98: (no net) -> +3.3V
- U1 pad 99: (no net) -> GND
Routing:
- net /HALT: track 64.9 -> 0.00 mm
- net /BUSREQ: track 60.5 -> 0.00 mm
- net /RESET: track 57.9 -> 0.00 mm
- net /INSTRD: track 55.3 -> 0.00 mm
- net /BUSACK: track 54.5 -> 0.00 mm
- net /RD: track 51.8 -> 0.00 mm
- net /NMI: track 51.0 -> 0.00 mm
- net /IORQ: track 49.3 -> 0.00 mm
- net /WAIT: track 48.5 -> 0.00 mm
- net N-0000018: track 46.9 -> 0.00 mm
- net N-0000019: track 46.3 -> 0.00 mm
- net /D6: track 45.8 -> 0.00 mm
- net N-0000047: track 15.4 -> 60.7 mm
- net N-0000020: track 45.3 -> 0.00 mm
- net /WR: track 45.0 -> 0.00 mm
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Other:
- net class Default: clearance 0.254 -> 0.199; trace_width 0.2032 -> 0.2; via_dia 0.889 -> 0.6; via_drill 0.635 -> 0.3
- rule trace_clearance: 0.254 -> 0.199
- rule trace_min: 0.2032 -> 0.15
- rule via_min_drill: 0.635 -> 0.3
- rule via_min_size: 0.889 -> 0.6
- board text removed: "3.3V"
- board text removed: "A0"
- board text removed: "A1"
- board text removed: "A10"
- board text removed: "A11"
- board text removed: "A12"
- board text removed: "A13"
- board text removed: "A14"
- board text removed: "A15"
- board text removed: "A16"
- board text removed: "A17"
- board text removed: "A18"
- board text removed: "A19"
- board text removed: "A2"
- board text removed: "A20"
- board text removed: "A22"
- board text removed: "A23"
- board text removed: "A3"
- board text removed: "A4"
- board text removed: "A5"
- board text removed: "A6"
- board text removed: "A7"
- board text removed: "A8"
- board text removed: "A9"
- board text removed: "ACK"
- board text removed: "CONTROL"
- board text removed: "CS"
- board text removed: "CS0"
- board text removed: "CS1"
- board text removed: "CS2"
- board text removed: "CS3"
- board text removed: "CTS"
- board text removed: "D0"
- board text removed: "D1"
- board text removed: "D2"
- board text removed: "D3"
- board text removed: "D4"
- board text removed: "D5"
- board text removed: "D6"
- board text removed: "D7"
- board text removed: "DCD"
- board text removed: "DSR"
- board text removed: "DTR"
- board text removed: "EC0"
- board text removed: "EC1"
- board text removed: "GND"
- board text removed: "HLT"
- board text removed: "IC1"
- board text removed: "IC2"
- board text removed: "IC3"
- board text removed: "INST"
- board text removed: "IORQ"
- board text removed: "MISO"
- board text removed: "MOSI"
- board text removed: "MRQ"
- board text removed: "NMI"
- board text removed: "NPWM3"
- board text removed: "OC0"
- board text removed: "OC1"
- board text removed: "OC2"
- board text removed: "OC3"
- board text removed: "RD"
- board text removed: "REQ"
- board text removed: "RES"
- board text removed: "RI"
- board text removed: "RTS"
- board text removed: "RXD"
- board text removed: "SCK"
- board text removed: "SS"
- board text removed: "TOUT0"
- board text removed: "TOUT2"
- board text removed: "TXD"
- board text removed: "WAIT"
- board text removed: "WP"
- board text removed: "WR"
